Commit message: 自駕OK

File: sensor_kit/sample_sensor_kit_launch/sample_sensor_kit_description/urdf/sensor_kit.xacro (robot description, xacro)
@@ -39,5 +39,5 @@
       pitch="${calibration['sensor_kit_base_link']['imu_link']['pitch']}"
       yaw="${calibration['sensor_kit_base_link']['imu_link']['yaw']}"
-      fps="100"
+      fps="400"
     />
   </xacro:macro>

File: vehicle/sample_vehicle_launch/sample_vehicle_description/urdf/vehicle.xacro (robot description, xacro)
@@ -8,5 +8,5 @@
       <origin xyz="${vehicle_info['/**']['ros__parameters']['wheel_base']/2.0} 0 0" rpy="${pi/2.0} 0 ${pi}"/>
       <geometry>
-        <mesh filename="package://sample_vehicle_description/mesh/lexus.dae" scale="1 1 1"/>
+        <mesh filename="package://sample_vehicle_description/mesh/lexus.dae" scale="0.5 0.5 0.5"/>
       </geometry>
     </visual>

Commit message: fix: clean up usb_cam launch without sensing/, override node commented

File: sensor_kit/sample_sensor_kit_launch/sample_sensor_kit_description/urdf/sensor_kit.xacro (robot description, xacro)
@@ -19,5 +19,5 @@
     <xacro:property name="calibration" value="${xacro.load_yaml('$(arg config_dir)/sensor_kit_calibration.yaml')}"/>
     <!-- lidar -->
-    <xacro:VLP-16 parent="sensor_kit_base_link" name="velodyne_top" topic="/points_raw" hz="10" samples="220" gpu="$(arg gpu)">
+    <xacro:VLP-16 parent="sensor_kit_base_link" name="velodyne_top" topic="/points_raw" hz="20" samples="220" gpu="$(arg gpu)">
       <origin
         xyz="${calibration['sensor_kit_base_link']['velodyne_top_base_link']['x']}
@@ -40,57 +40,55 @@
       pitch="${calibration['sensor_kit_base_link']['imu_link']['pitch']}"
       yaw="${calibration['sensor_kit_base_link']['imu_link']['yaw']}"
-      fps="400"
+      fps="200"
     />
     <!-- camera_f -->
     <!-- camera 0 (前方) -->
   <xacro:monocular_camera_macro
-    name="camera/camera0/camera"
+    name="camera_f/camera"
     parent="sensor_kit_base_link"
     namespace=""
-    x="${calibration['sensor_kit_base_link']['camera/camera0/camera_link']['x']}"
-    y="${calibration['sensor_kit_base_link']['camera/camera0/camera_link']['y']}"
-    z="${calibration['sensor_kit_base_link']['camera/camera0/camera_link']['z']}"
-    roll="${calibration['sensor_kit_base_link']['camera/camera0/camera_link']['roll']}"
-    pitch="${calibration['sensor_kit_base_link']['camera/camera0/camera_link']['pitch']}"
-    yaw="${calibration['sensor_kit_base_link']['camera/camera0/camera_link']['yaw']}"
+    x="${calibration['sensor_kit_base_link']['camera_f/camera_link']['x']}"
+    y="${calibration['sensor_kit_base_link']['camera_f/camera_link']['y']}"
+    z="${calibration['sensor_kit_base_link']['camera_f/camera_link']['z']}"
+    roll="${calibration['sensor_kit_base_link']['camera_f/camera_link']['roll']}"
+    pitch="${calibration['sensor_kit_base_link']['camera_f/camera_link']['pitch']}"
+    yaw="${calibration['sensor_kit_base_link']['camera_f/camera_link']['yaw']}"
     fps="30" width="1920" height="1080" fov="1.3"
   />
   <!-- camera 1 (後方) -->
   <xacro:monocular_camera_macro
-    name="camera/camera1/camera"
+    name="camera_b/camera"
     parent="sensor_kit_base_link"
     namespace=""
-    x="${calibration['sensor_kit_base_link']['camera/camera1/camera_link']['x']}"
-    y="${calibration['sensor_kit_base_link']['camera/camera1/camera_link']['y']}"
-    z="${calibration['sensor_kit_base_link']['camera/camera1/camera_link']['z']}"
-    roll="${calibration['sensor_kit_base_link']['camera/camera1/camera_link']['roll']}"
-    pitch="${calibration['sensor_kit_base_link']['camera/camera1/camera_link']['pitch']}"
-    yaw="${calibration['sensor_kit_base_link']['camera/camera1/camera_link']['yaw']}"
+    x="${calibration['sensor_kit_base_link']['camera_b/camera_link']['x']}"
+    y="${calibration['sensor_kit_base_link']['camera_b/camera_link']['y']}"
+    z="${calibration['sensor_kit_base_link']['camera_b/camera_link']['z']}"
+    roll="${calibration['sensor_kit_base_link']['camera_b/camera_link']['roll']}"
+    pitch="${calibration['sensor_kit_base_link']['camera_b/camera_link']['pitch']}"
+    yaw="${calibration['sensor_kit_base_link']['camera_b/camera_link']['yaw']}"
     fps="30" width="1920" height="1080" fov="1.3"
   />
-  <!-- camera 2 (右方) -->
   <xacro:monocular_camera_macro
-    name="camera/camera2/camera"
+    name="camera_l/camera"
     parent="sensor_kit_base_link"
     namespace=""
-    x="${calibration['sensor_kit_base_link']['camera/camera2/camera_link']['x']}"
-    y="${calibration['sensor_kit_base_link']['camera/camera2/camera_link']['y']}"
-    z="${calibration['sensor_kit_base_link']['camera/camera2/camera_link']['z']}"
-    roll="${calibration['sensor_kit_base_link']['camera/camera2/camera_link']['roll']}"
-    pitch="${calibration['sensor_kit_base_link']['camera/camera2/camera_link']['pitch']}"
-    yaw="${calibration['sensor_kit_base_link']['camera/camera2/camera_link']['yaw']}"
+    x="${calibration['sensor_kit_base_link']['camera_l/camera_link']['x']}"
+    y="${calibration['sensor_kit_base_link']['camera_l/camera_link']['y']}"
+    z="${calibration['sensor_kit_base_link']['camera_l/camera_link']['z']}"
+    roll="${calibration['sensor_kit_base_link']['camera_l/camera_link']['roll']}"
+    pitch="${calibration['sensor_kit_base_link']['camera_l/camera_link']['pitch']}"
+    yaw="${calibration['sensor_kit_base_link']['camera_l/camera_link']['yaw']}"
     fps="30" width="1920" height="1080" fov="1.3"
   />
-  <!-- camera 3 (左方) -->
   <xacro:monocular_camera_macro
-    name="camera/camera3/camera"
+    name="camera_r/camera"
     parent="sensor_kit_base_link"
     namespace=""
-    x="${calibration['sensor_kit_base_link']['camera/camera3/camera_link']['x']}"
-    y="${calibration['sensor_kit_base_link']['camera/camera3/camera_link']['y']}"
-    z="${calibration['sensor_kit_base_link']['camera/camera3/camera_link']['z']}"
-    roll="${calibration['sensor_kit_base_link']['camera/camera3/camera_link']['roll']}"
-    pitch="${calibration['sensor_kit_base_link']['camera/camera3/camera_link']['pitch']}"
-    yaw="${calibration['sensor_kit_base_link']['camera/camera3/camera_link']['yaw']}"
+    x="${calibration['sensor_kit_base_link']['camera_r/camera_link']['x']}"
+    y="${calibration['sensor_kit_base_link']['camera_r/camera_link']['y']}"
+    z="${calibration['sensor_kit_base_link']['camera_r/camera_link']['z']}"
+    roll="${calibration['sensor_kit_base_link']['camera_r/camera_link']['roll']}"
+    pitch="${calibration['sensor_kit_base_link']['camera_r/camera_link']['pitch']}"
+    yaw="${calibration['sensor_kit_base_link']['camera_r/camera_link']['yaw']}"
     fps="30" width="1920" height="1080" fov="1.3"
   />

File: vehicle/sample_vehicle_launch/sample_vehicle_description/urdf/vehicle.xacro (robot description, xacro)
@@ -8,5 +8,5 @@
       <origin xyz="${vehicle_info['/**']['ros__parameters']['wheel_base']/2.0} 0 0" rpy="${pi/2.0} 0 ${pi}"/>
       <geometry>
-        <mesh filename="package://sample_vehicle_description/mesh/lexus.dae" scale="0.5 0.5 0.5"/>
+        <mesh filename="package://sample_vehicle_description/mesh/lexus.dae" scale="0.4 0.4 0.4"/>
       </geometry>
     </visual>
